Commit message: fixed a height offset issue

File: urdf/velodyne.urdf.xacro (robot description, xacro)
@@ -65,5 +65,5 @@
   <joint name="velodyne_spindle" type="continuous">
     <axis xyz="0 1 0" />
-    <origin xyz="0 0 0" rpy="1.57 0 0"/>
+    <origin xyz="0 0 0.1" rpy="1.57 0 0"/>
     <parent link="velodyne_laser_static"/>
     <child link="velodyne_laser_spin"/>
@@ -127,5 +127,5 @@
                reading. -->
           <mean>0.0</mean>
-          <stddev>0.01</stddev>
+          <stddev>0.0</stddev>
         </noise>
       </ray>
